Commit message: --

File: install/robotic_arm_moveit_config/share/robotic_arm_moveit_config/config/robotic_arm.ros2_control.xacro (robot description, xacro)
@@ -1,113 +1 @@
-<?xml version="1.0"?>
-<robot xmlns:xacro="http://www.ros.org/wiki/xacro">
-  <xacro:macro name="robotic_arm_ros2_control" params="name initial_positions_file">
-    <xacro:property name="initial_positions" value="${xacro.load_yaml(initial_positions_file)['initial_positions']}"/>
-    <ros2_control name="${name}" type="system">
-      <hardware>
-        <plugin>mock_components/GenericSystem</plugin>
-        <param name="command_interfaces">
-          position
-        </param>
-        <param name="state_interfaces">
-          position
-          velocity
-        </param>
-      </hardware>
-      <joint name="rotating_base_joint">
-        <command_interface name="position"/>
-        <state_interface name="position">
-          <param name="initial_value">${initial_positions['rotating_base_joint']}</param>
-        </state_interface>
-        <state_interface name="velocity"/>
-      </joint>
-      <joint name="shoulder_joint">
-        <command_interface name="position"/>
-        <state_interface name="position">
-          <param name="initial_value">${initial_positions['shoulder_joint']}</param>
-        </state_interface>
-        <state_interface name="velocity"/>
-      </joint>
-      <joint name="elbow_joint">
-        <command_interface name="position"/>
-        <state_interface name="position">
-          <param name="initial_value">${initial_positions['elbow_joint']}</param>
-        </state_interface>
-        <state_interface name="velocity"/>
-      </joint>
-      <joint name="forearm_joint">
-        <command_interface name="position"/>
-        <state_interface name="position">
-          <param name="initial_value">${initial_positions['forearm_joint']}</param>
-        </state_interface>
-        <state_interface name="velocity"/>
-      </joint>
-      <joint name="wrist_joint">
-        <command_interface name="position"/>
-        <state_interface name="position">
-          <param name="initial_value">${initial_positions['wrist_joint']}</param>
-        </state_interface>
-        <state_interface name="velocity"/>
-      </joint>
-      <joint name="gripper_right_joint">
-        <command_interface name="position"/>
-        <state_interface name="position">
-          <param name="initial_value">${initial_positions['gripper_right_joint']}</param>
-        </state_interface>
-        <state_interface name="velocity"/>
-      </joint>
-    </ros2_control>
-  </xacro:macro>
-</robot>
-<!-- <?xml version="1.0"?>
-<robot xmlns:xacro="http://www.ros.org/wiki/xacro">
-    <xacro:macro name="robotic_arm_ros2_control" params="name initial_positions_file">
-        <xacro:property name="initial_positions" value="${xacro.load_yaml(initial_positions_file)['initial_positions']}"/>
-        <ros2_control name="${name}" type="system">
-            <hardware>
-                <plugin>mock_components/GenericSystem</plugin>
-            </hardware>
-            <joint name="rotating_base_joint">
-                <command_interface name="position"/>
-                <state_interface name="position">
-                  <param name="initial_value">${initial_positions['rotating_base_joint']}</param>
-                </state_interface>
-                <state_interface name="velocity"/>
-            </joint>
-            <joint name="shoulder_joint">
-                <command_interface name="position"/>
-                <state_interface name="position">
-                  <param name="initial_value">${initial_positions['shoulder_joint']}</param>
-                </state_interface>
-                <state_interface name="velocity"/>
-            </joint>
-            <joint name="elbow_joint">
-                <command_interface name="position"/>
-                <state_interface name="position">
-                  <param name="initial_value">${initial_positions['elbow_joint']}</param>
-                </state_interface>
-                <state_interface name="velocity"/>
-            </joint>
-            <joint name="forearm_joint">
-                <command_interface name="position"/>
-                <state_interface name="position">
-                  <param name="initial_value">${initial_positions['forearm_joint']}</param>
-                </state_interface>
-                <state_interface name="velocity"/>
-            </joint>
-            <joint name="wrist_joint">
-                <command_interface name="position"/>
-                <state_interface name="position">
-                  <param name="initial_value">${initial_positions['wrist_joint']}</param>
-                </state_interface>
-                <state_interface name="velocity"/>
-            </joint>
-            <joint name="gripper_right_joint">
-                <command_interface name="position"/>
-                <state_interface name="position">
-                  <param name="initial_value">${initial_positions['gripper_right_joint']}</param>
-                </state_interface>
-                <state_interface name="velocity"/>
-            </joint>
-        </ros2_control>
-    </xacro:macro>
-</robot> -->
+/home/saber/robox_ws/src/robotic_arm_moveit_config/config/robotic_arm.ros2_control.xacro

File: install/robotic_arm_moveit_config/share/robotic_arm_moveit_config/config/robotic_arm.urdf.xacro (robot description, xacro)
@@ -1,12 +1 @@
-<?xml version="1.0"?>
-<robot xmlns:xacro="http://www.ros.org/wiki/xacro" name="robotic_arm">
-    <xacro:arg name="initial_positions_file" default="initial_positions.yaml" />
-    <xacro:include filename="$(find arm_description)/urdf/arm.urdf" />
-    <xacro:include filename="robotic_arm.ros2_control.xacro" />
-    <visual>
-  <geometry>
-    <mesh filename="package://arm_description/meshes/base_link.stl"/>
-  </geometry>
-</visual>
-    <xacro:robotic_arm_ros2_control name="FakeSystem" initial_positions_file="$(arg initial_positions_file)"/>
-</robot>
+/home/saber/robox_ws/src/robotic_arm_moveit_config/config/robotic_arm.urdf.xacro

File: install/robotic_arm_moveit_config/share/robotic_arm_moveit_config/config/ros2_control.xacro (robot description, xacro)
@@ -1,73 +1 @@
-<?xml version="1.0"?>
-<robot xmlns:xacro="http://www.ros.org/wiki/xacro">
-  <xacro:macro name="robotic_arm_ros2_control" params="name initial_positions_file">
-    <xacro:property name="initial_positions" value="${xacro.load_yaml(initial_positions_file)['initial_positions']}"/>
-    <ros2_control name="${name}" type="system">
-      <hardware>
-        <plugin>mock_components/GenericSystem</plugin>
-        <param name="mock_sensor_commands">false</param>
-        <param name="state_following_offset">0.0</param>
-      </hardware>
-      <joint name="rotating_base_joint">
-        <command_interface name="position">
-          <param name="min">-1.57</param>
-          <param name="max">1.22</param>
-        </command_interface>
-        <state_interface name="position">
-          <param name="initial_value">${initial_positions['rotating_base_joint']}</param>
-        </state_interface>
-        <state_interface name="velocity"/>
-      </joint>
-      <joint name="shoulder_joint">
-        <command_interface name="position">
-          <param name="min">-1.308</param>
-          <param name="max">0.61</param>
-        </command_interface>
-        <state_interface name="position">
-          <param name="initial_value">${initial_positions['shoulder_joint']}</param>
-        </state_interface>
-        <state_interface name="velocity"/>
-      </joint>
-      <joint name="elbow_joint">
-        <command_interface name="position">
-          <param name="min">-1.57</param>
-          <param name="max">1.57</param>
-        </command_interface>
-        <state_interface name="position">
-          <param name="initial_value">${initial_positions['elbow_joint']}</param>
-        </state_interface>
-        <state_interface name="velocity"/>
-      </joint>
-      <joint name="forearm_joint">
-        <command_interface name="position">
-          <param name="min">-1.57</param>
-          <param name="max">1.57</param>
-        </command_interface>
-        <state_interface name="position">
-          <param name="initial_value">${initial_positions['forearm_joint']}</param>
-        </state_interface>
-        <state_interface name="velocity"/>
-      </joint>
-      <joint name="wrist_joint">
-        <command_interface name="position">
-          <param name="min">-1.57</param>
-          <param name="max">1.57</param>
-        </command_interface>
-        <state_interface name="position">
-          <param name="initial_value">${initial_positions['wrist_joint']}</param>
-        </state_interface>
-        <state_interface name="velocity"/>
-      </joint>
-      <joint name="gripper_right_joint">
-        <command_interface name="position">
-          <param name="min">0.0</param>
-          <param name="max">0.8</param>
-        </command_interface>
-        <state_interface name="position">
-          <param name="initial_value">${initial_positions['gripper_right_joint']}</param>
-        </state_interface>
-        <state_interface name="velocity"/>
-      </joint>
-    </ros2_control>
-  </xacro:macro>
-</robot>
+/home/saber/robox_ws/src/robotic_arm_moveit_config/config/ros2_control.xacro

File: install/robotic_arm_moveit_config/share/robotic_arm_moveit_config/config/urdf/robotic_arm.urdf.xacro (robot description, xacro)
@@ -1,356 +1 @@
-<?xml version="1.0" encoding="utf-8"?>
-<robot name="robotic_arm">
-  <!-- Material Definitions -->
-  <material name="blue">
-    <color rgba="0.0 0.0 0.8 1"/>
-  </material>
-  <material name="silver">
-    <color rgba="0.75 0.75 0.75 1"/>
-  </material>
-  <!-- World Link -->
-  <link name="world"/>
-  <!-- Base Joint -->
-  <joint name="world_to_base" type="fixed">
-    <parent link="world"/>
-    <child link="base_link"/>
-    <origin xyz="0 0 0" rpy="1.5 1.5 1.5"/>
-  </joint>
-  <!-- Base Link -->
-  <link name="base_link">
-    <inertial>
-      <origin xyz="-0.035398 -0.0004353 0.027453" rpy="0 0 0"/>
-      <mass value="0.39671"/>
-      <inertia
-        ixx="0.00092742"
-        ixy="-4.6465E-07"
-        ixz="3.0759E-08"
-        iyy="0.00057216"
-        iyz="1.5079E-07"
-        izz="0.00037377"/>
-    </inertial>
-    <visual>
-      <origin xyz="0 0 0" rpy="0 0 0"/>
-      <geometry>
-        <mesh filename="package://arm_description/meshes/base_link.STL"/>
-      </geometry>
-      <material name="blue"/>
-    </visual>
-    <collision>
-      <origin xyz="0 0 0" rpy="0 0 0"/>
-      <geometry>
-        <mesh filename="package://arm_description/meshes/base_link.STL"/>
-      </geometry>
-    </collision>
-  </link>
-  <!-- Rotating Base Link -->
-  <link name="rotating_base_link">
-    <inertial>
-      <origin xyz="0.000158275887253499 0.027492254844178 -0.00611871263232042" rpy="0 0 0"/>
-      <mass value="0.0561612792514196"/>
-      <inertia
-        ixx="9.9128401791064E-06"
-        ixy="2.12663345089064E-11"
-        ixz="3.39707661438049E-08"
-        iyy="1.76973775421821E-05"
-        iyz="4.60310716010097E-07"
-        izz="1.32217491388007E-05"/>
-    </inertial>
-    <visual>
-      <origin xyz="0 0 0" rpy="0 0 0"/>
-      <geometry>
-        <mesh filename="package://arm_description/meshes/rotating_base_link.STL"/>
-      </geometry>
-      <material name="blue"/>
-    </visual>
-    <collision>
-      <origin xyz="0 0 0" rpy="0 0 0"/>
-      <geometry>
-        <mesh filename="package://arm_description/meshes/rotating_base_link.STL"/>
-      </geometry>
-    </collision>
-  </link>
-  <!-- Rotating Base Joint -->
-  <joint name="rotating_base_joint" type="revolute">
-    <origin xyz="-0.0466999999999999 0 0" rpy="0 -1.52754450035515 1.5707963267949"/>
-    <parent link="base_link"/>
-    <child link="rotating_base_link"/>
-    <axis xyz="0 1 0"/>
-    <limit lower="-1.57" upper="1.220" effort="100" velocity="2"/>
-  </joint>
-  <!-- Shoulder Link -->
-  <link name="shoulder_link">
-    <inertial>
-      <origin xyz="0.05 0.00141746277739371 -0.00395375026056261" rpy="0 0 0"/>
-      <mass value="0.0422835365975949"/>
-      <inertia
-        ixx="2.5539223828081E-05"
-        ixy="5.2304284492953E-20"
-        ixz="5.09708693455176E-21"
-        iyy="3.9772332084034E-05"
-        iyz="-6.979081923206E-08"
-        izz="5.89921114741114E-05"/>
-    </inertial>
-    <visual>
-      <origin xyz="0 0 0" rpy="0 0 0"/>
-      <geometry>
-        <mesh filename="package://arm_description/meshes/shoulder_link.STL"/>
-      </geometry>
-      <material name="blue"/>
-    </visual>
-    <collision>
-      <origin xyz="0 0 0" rpy="0 0 0"/>
-      <geometry>
-        <mesh filename="package://arm_description/meshes/shoulder_link.STL"/>
-      </geometry>
-    </collision>
-  </link>
-  <!-- Shoulder Joint -->
-  <joint name="shoulder_joint" type="revolute">
-    <origin xyz="-0.00949999999999954 0.0308700000000001 0" rpy="-1.5 0 1.5"/>
-    <parent link="rotating_base_link"/>
-    <child link="shoulder_link"/>
-    <axis xyz="0 1 0"/>
-    <limit lower="-1.308" upper="0.610" effort="100" velocity="2"/>
-  </joint>
-  <!-- Elbow Link -->
-  <link name="elbow_link">
-    <inertial>
-      <origin xyz="-0.0450025328071686 -0.0042809747594438 -0.00130547754639812" rpy="0 0 0"/>
-      <mass value="0.13493321141733"/>
-      <inertia
-        ixx="3.06279251143249E-05"
-        ixy="1.20337731418417E-09"
-        ixz="-1.91215180545226E-09"
-        iyy="8.18401391205364E-05"
-        iyz="1.06896103680731E-06"
-        izz="0.000101277084508677"/>
-    </inertial>
-    <visual>
-      <origin xyz="0 0 0" rpy="0 0 0"/>
-      <geometry>
-        <mesh filename="package://arm_description/meshes/elbow_link.STL"/>
-      </geometry>
-      <material name="blue"/>
-    </visual>
-    <collision>
-      <origin xyz="0 0 0" rpy="0 0 0"/>
-      <geometry>
-        <mesh filename="package://arm_description/meshes/elbow_link.STL"/>
-      </geometry>
-    </collision>
-  </link>
-  <!-- Elbow Joint -->
-  <joint name="elbow_joint" type="revolute">
-    <origin xyz="0.1 0 0" rpy="0 0.080837952 3.14159265358978"/>
-    <parent link="shoulder_link"/>
-    <child link="elbow_link"/>
-    <axis xyz="0 1 0"/>
-    <limit lower="-1.57" upper="1.57" effort="100" velocity="2"/>
-  </joint>
-  <!-- Forearm Link -->
-  <link name="forearm_link">
-    <inertial>
-      <origin xyz="0.0010832320248741 -0.047774444639081 -0.000231064174041173" rpy="0 0 0"/>
-      <mass value="0.0447180559582269"/>
-      <inertia
-        ixx="1.67225851396217E-05"
-        ixy="-1.16841164754521E-07"
-        ixz="-2.11846893656155E-11"
-        iyy="1.4108277215624E-05"
-        iyz="-3.39709530009559E-08"
-        izz="1.67748719855516E-05"/>
-    </inertial>
-    <visual>
-      <origin xyz="0 0 0" rpy="0 0 0"/>
-      <geometry>
-        <mesh filename="package://arm_description/meshes/forearm_link.STL"/>
-      </geometry>
-      <material name="blue"/>
-    </visual>
-    <collision>
-      <origin xyz="0 0 0" rpy="0 0 0"/>
-      <geometry>
-        <mesh filename="package://arm_description/meshes/forearm_link.STL"/>
-      </geometry>
-    </collision>
-  </link>
-  <!-- Forearm Joint -->
-  <joint name="forearm_joint" type="revolute">
-    <origin xyz="-0.0899999999999956 0 0" rpy="0.040178506 0 -1.57079632679489"/>
-    <parent link="elbow_link"/>
-    <child link="forearm_link"/>
-    <axis xyz="1 0 0"/>
-    <limit lower="-1.57" upper="1.57" effort="100" velocity="2"/>
-  </joint>
-  <!-- Wrist Link -->
-  <link name="wrist_link">
-    <inertial>
-      <origin xyz="0.0190989125713327 0.00061469939040844 0.00252312799008259" rpy="0 0 0"/>
-      <mass value="0.0529522848326195"/>
-      <inertia
-        ixx="1.10404885697885E-05"
-        ixy="-1.53962728731698E-07"
-        ixz="-9.76735867241465E-07"
-        iyy="1.00687044394914E-05"
-        iyz="-3.98653063319089E-07"
-        izz="1.82604593599498E-05"/>
-    </inertial>
-    <visual>
-      <origin xyz="0 0 0" rpy="0 0 0"/>
-      <geometry>
-        <mesh filename="package://arm_description/meshes/wrist_link.STL"/>
-      </geometry>
-      <material name="silver"/>
-    </visual>
-    <collision>
-      <origin xyz="0 0 0" rpy="0 0 0"/>
-      <geometry>
-        <mesh filename="package://arm_description/meshes/wrist_link.STL"/>
-      </geometry>
-    </collision>
-  </link>
-  <!-- Wrist Joint -->
-  <joint name="wrist_joint" type="revolute">
-    <origin xyz="0.00099999999999714 -0.0795710619584145 -0.0097500000000017" rpy="-3.1124530411889 0 -1.5707963267949"/>
-    <parent link="forearm_link"/>
-    <child link="wrist_link"/>
-    <axis xyz="1 0 0"/>
-    <limit lower="-1.57" upper="1.57" effort="100" velocity="2"/>
-  </joint>
-  <!-- Gripper Left Link -->
-  <link name="gripper_left_link">
-    <inertial>
-      <origin xyz="0.0484172860271485 -0.0241584658945902 0.0142380102355266" rpy="0 0 0"/>
-      <mass value="0.0163529802377136"/>
-      <inertia
-        ixx="2.95937890453479E-06"
-        ixy="1.60740985116118E-06"
-        ixz="4.04413653565078E-09"
-        iyy="2.27972601870315E-06"
-        iyz="1.56748388623883E-12"
-        izz="4.68843868201044E-06"/>
-    </inertial>
-    <visual>
-      <origin xyz="0 0 0" rpy="0 0 0"/>
-      <geometry>
-        <mesh filename="package://arm_description/meshes/gripper_left_link.STL"/>
-      </geometry>
-      <material name="silver"/>
-    </visual>
-    <collision>
-      <origin xyz="0 0 0" rpy="0 0 0"/>
-      <geometry>
-        <mesh filename="package://arm_description/meshes/gripper_left_link.STL"/>
-      </geometry>
-    </collision>
-  </link>
-  <!-- Gripper Left Joint -->
-  <joint name="gripper_left_joint" type="revolute">
-    <origin xyz="0.031104 0 0" rpy="0.023878 -0.042377 1.0575"/>
-    <parent link="wrist_link"/>
-    <child link="gripper_left_link"/>
-    <axis xyz="0 0 1"/>
-    <limit lower="-1.57" upper="1.57" effort="100" velocity="2"/>
-    <mimic joint="gripper_right_joint" multiplier="1" offset="0"/>
-  </joint>
-  <!-- Gripper Right Link -->
-  <link name="gripper_right_link">
-    <inertial>
-      <origin xyz="-0.0375860640609017 -0.0369591692006576 -0.0142262545696464" rpy="0 0 0"/>
-      <mass value="0.016328263992727"/>
-      <inertia
-        ixx="1.31332905769687E-06"
-        ixy="-9.9717065345883E-07"
-        ixz="1.4036038701819E-09"
-        iyy="3.92463290581539E-06"
-        iyz="3.79932405367648E-09"
-        izz="4.68749882724247E-06"/>
-    </inertial>
-    <visual>
-      <origin xyz="0 0 0" rpy="0 0 0"/>
-      <geometry>
-        <mesh filename="package://arm_description/meshes/gripper_right_link.STL"/>
-      </geometry>
-      <material name="silver"/>
-    </visual>
-    <collision>
-      <origin xyz="0 0 0" rpy="0 0 0"/>
-      <geometry>
-        <mesh filename="package://arm_description/meshes/gripper_right_link.STL"/>
-      </geometry>
-    </collision>
-  </link>
-  <!-- Gripper Right Joint -->
-  <joint name="gripper_right_joint" type="revolute">
-    <origin xyz="0.033035 0 0" rpy="3.0936 0.0076308 -2.9842"/>
-    <parent link="wrist_link"/>
-    <child link="gripper_right_link"/>
-    <axis xyz="0 0 1"/>
-    <limit lower="-1.57" upper="1.57" effort="100" velocity="2"/>
-  </joint>
-  <!-- ROS2 Control -->
-  <ros2_control name="RobotControl" type="system">
-    <hardware>
-<plugin>mock_components/GenericSystem</plugin>
-      <param name="state_following_offset">0.0</param>
-    </hardware>
-    <joint name="rotating_base_joint">
-      <command_interface name="position">
-        <param name="min">-1.57</param>
-        <param name="max">1.220</param>
-      </command_interface>
-      <state_interface name="position"/>
-      <state_interface name="velocity"/>
-    </joint>
-    <joint name="shoulder_joint">
-      <command_interface name="position">
-        <param name="min">-1.308</param>
-        <param name="max">0.610</param>
-      </command_interface>
-      <state_interface name="position"/>
-      <state_interface name="velocity"/>
-    </joint>
-    <joint name="elbow_joint">
-      <command_interface name="position">
-        <param name="min">-1.57</param>
-        <param name="max">1.57</param>
-      </command_interface>
-      <state_interface name="position"/>
-      <state_interface name="velocity"/>
-    </joint>
-    <joint name="forearm_joint">
-      <command_interface name="position">
-        <param name="min">-1.57</param>
-        <param name="max">1.57</param>
-      </command_interface>
-      <state_interface name="position"/>
-      <state_interface name="velocity"/>
-    </joint>
-    <joint name="wrist_joint">
-      <command_interface name="position">
-        <param name="min">-1.57</param>
-        <param name="max">1.57</param>
-      </command_interface>
-      <state_interface name="position"/>
-      <state_interface name="velocity"/>
-    </joint>
-    <!-- Gripper joints -->
-    <joint name="gripper_right_joint">
-      <command_interface name="position">
-        <param name="min">-1.221</param>
-        <param name="max">0.097</param>
-      </command_interface>
-      <state_interface name="position"/>
-      <state_interface name="velocity"/>
-    </joint>
-    <!-- Optional: Keep gripper_left_joint if needed but not controlled -->
-    <!-- <joint name="gripper_left_joint">
-      <command_interface name="position">
-        <param name="min">-1.57</param>
-        <param name="max">1.57</param>
-      </command_interface>
-      <state_interface name="position"/>
-      <state_interface name="velocity"/>
-    </joint> -->
-  </ros2_control>
-</robot>
+/home/saber/robox_ws/src/robotic_arm_moveit_config/config/urdf/robotic_arm.urdf.xacro

File: src/arm_description/urdf/arm.urdf (robot description, URDF)
Before this commit: robot robotic_arm, 9 links, 8 joints
Links:
- removed link world
Joints:
- removed joint world_to_base
