Commit message: fixe ik problems & editing the urdf

File: install/moveit_resources_prbt_support/share/moveit_resources_prbt_support/urdf/prbt.ros2_control.xacro (robot description, xacro)
@@ -1 +1,134 @@
-/home/saber/robox_ws/src/moveit2/moveit_planners/test_configs/prbt_support/urdf/prbt.ros2_control.xacro
+<?xml version="1.0"?>
+<robot xmlns:xacro="http://www.ros.org/wiki/xacro">
+	<xacro:macro name="prbt_ros2_control" params="name prefix use_fake_hardware:=true fake_sensor_commands:=true initial_positions">
+		<ros2_control name="${name}" type="system">
+			<hardware>
+				<xacro:if value="${use_fake_hardware}">
+					<plugin>mock_components/GenericSystem</plugin>
+					<param name="fake_sensor_commands">${fake_sensor_commands}</param>
+					<param name="state_following_offset">0.0</param>
+				</xacro:if>
+			</hardware>
+			<joint name="${prefix}joint_1">
+				<command_interface name="position">
+					<param name="min">-2.96706</param>
+					<param name="max">2.96706</param>
+				</command_interface>
+				<command_interface name="velocity">
+					<param name="min">-3.15</param>
+					<param name="max">3.15</param>
+				</command_interface>
+				<state_interface name="position">
+					<param name="initial_value">0.0</param>
+				</state_interface>
+				<state_interface name="velocity">
+					<param name="initial_value">0.0</param>
+				</state_interface>
+				<state_interface name="effort">
+					<param name="initial_value">0.0</param>
+				</state_interface>
+				<param name="initial_position">${initial_positions['joint_1']}</param>  <!-- initial position for the FakeSystem -->
+			</joint>
+			<joint name="${prefix}joint_2">
+				<command_interface name="position">
+					<param name="min">-2.96706</param>
+					<param name="max">2.96706</param>
+				</command_interface>
+				<command_interface name="velocity">
+					<param name="min">-3.15</param>
+					<param name="max">3.15</param>
+				</command_interface>
+				<state_interface name="position">
+					<param name="initial_value">0.0</param>
+				</state_interface>
+				<state_interface name="velocity">
+					<param name="initial_value">0.0</param>
+				</state_interface>
+				<state_interface name="effort">
+					<param name="initial_value">0.0</param>
+				</state_interface>
+				<param name="initial_position">${initial_positions['joint_2']}</param>  <!-- initial position for the FakeSystem -->
+			</joint>
+			<joint name="${prefix}joint_3">
+				<command_interface name="position">
+					<param name="min">-2.96706</param>
+					<param name="max">2.96706</param>
+				</command_interface>
+				<command_interface name="velocity">
+					<param name="min">-3.15</param>
+					<param name="max">3.15</param>
+				</command_interface>
+				<state_interface name="position">
+					<param name="initial_value">0.0</param>
+				</state_interface>
+				<state_interface name="velocity">
+					<param name="initial_value">0.0</param>
+				</state_interface>
+				<state_interface name="effort">
+					<param name="initial_value">0.0</param>
+				</state_interface>
+				<param name="initial_position">${initial_positions['joint_3']}</param>  <!-- initial position for the FakeSystem -->
+			</joint>
+			<joint name="${prefix}joint_4">
+				<command_interface name="position">
+					<param name="min">-2.96706</param>
+					<param name="max">2.96706</param>
+				</command_interface>
+				<command_interface name="velocity">
+					<param name="min">-3.15</param>
+					<param name="max">3.15</param>
+				</command_interface>
+				<state_interface name="position">
+					<param name="initial_value">0.0</param>
+				</state_interface>
+				<state_interface name="velocity">
+					<param name="initial_value">0.0</param>
+				</state_interface>
+				<state_interface name="effort">
+					<param name="initial_value">0.0</param>
+				</state_interface>
+				<param name="initial_position">${initial_positions['joint_4']}</param>  <!-- initial position for the FakeSystem -->
+			</joint>
+			<joint name="${prefix}joint_5">
+				<command_interface name="position">
+					<param name="min">-2.96706</param>
+					<param name="max">2.96706</param>
+				</command_interface>
+				<command_interface name="velocity">
+					<param name="min">-3.15</param>
+					<param name="max">3.15</param>
+				</command_interface>
+				<state_interface name="position">
+					<param name="initial_value">0.0</param>
+				</state_interface>
+				<state_interface name="velocity">
+					<param name="initial_value">0.0</param>
+				</state_interface>
+				<state_interface name="effort">
+					<param name="initial_value">0.0</param>
+				</state_interface>
+				<param name="initial_position">${initial_positions['joint_5']}</param>  <!-- initial position for the FakeSystem -->
+			</joint>
+			<joint name="${prefix}joint_6">
+				<command_interface name="position">
+					<param name="min">-2.96706</param>
+					<param name="max">2.96706</param>
+				</command_interface>
+				<command_interface name="velocity">
+					<param name="min">-3.15</param>
+					<param name="max">3.15</param>
+				</command_interface>
+				<state_interface name="position">
+					<param name="initial_value">0.0</param>
+				</state_interface>
+				<state_interface name="velocity">
+					<param name="initial_value">0.0</param>
+				</state_interface>
+				<state_interface name="effort">
+					<param name="initial_value">0.0</param>
+				</state_interface>
+				<param name="initial_position">${initial_positions['joint_6']}</param>  <!-- initial position for the FakeSystem -->
+			</joint>
+		</ros2_control>
+	</xacro:macro>
+</robot>

File: install/moveit_resources_prbt_support/share/moveit_resources_prbt_support/urdf/prbt.xacro (robot description, xacro)
@@ -1 +1,56 @@
-/home/saber/robox_ws/src/moveit2/moveit_planners/test_configs/prbt_support/urdf/prbt.xacro
+<?xml version="1.0" encoding="utf-8" ?>
+<!--
+Copyright (c) 2018 Pilz GmbH & Co. KG
+Licensed under the Apache License, Version 2.0 (the "License");
+you may not use this file except in compliance with the License.
+You may obtain a copy of the License at
+    http://www.apache.org/licenses/LICENSE-2.0
+Unless required by applicable law or agreed to in writing, software
+distributed under the License is distributed on an "AS IS" BASIS,
+WITHOUT WARRANTIES OR CONDITIONS OF ANY KIND, either express or implied.
+See the License for the specific language governing permissions and
+limitations under the License.
+-->
+<robot name="prbt" xmlns:xacro="http://www.ros.org/wiki/xacro">
+  <!-- Definition of robot name -->
+  <xacro:arg name="robot_prefix" default="prbt_"/>
+  <!-- macro definition of pilz lwa -->
+  <xacro:include filename="$(find moveit_resources_prbt_support)/urdf/prbt_macro.xacro" />
+  <!-- gripper -->
+  <xacro:arg name="gripper" default=""/>
+  <xacro:property name="gripper" value="$(arg gripper)"/>
+  <!-- TCP Offset -->
+  <xacro:if value="${not gripper}">
+    <xacro:arg name="tcp_offset_xyz" default="0 0 0"/>
+    <xacro:arg name="tcp_offset_rpy" default="0 0 0"/>
+  </xacro:if>
+  <xacro:if value="${gripper != ''}">
+    <xacro:include filename="$(find moveit_resources_prbt_${gripper}_support)/config/${gripper}_tcp_offset.xacro" />
+  </xacro:if>
+  <!-- instantiate the robot -->
+  <xacro:prbt prefix="$(arg robot_prefix)" />
+  <link name="world"/>
+  <joint name="world-base_link-fixed" type="fixed">
+    <parent link="world"/>
+    <child link="$(arg robot_prefix)base_link"/>
+  </joint>
+  <!-- TCP -->
+  <joint name="$(arg robot_prefix)fixed_joint_tcp" type="fixed">
+    <origin xyz="$(arg tcp_offset_xyz)" rpy="$(arg tcp_offset_rpy)" />  <!-- tcp offset from last link -->
+    <parent link="$(arg robot_prefix)flange"/>
+    <child link="$(arg robot_prefix)tcp"/>
+  </joint>
+  <link name="$(arg robot_prefix)tcp" />
+  <!-- If gripper given then... -->
+  <xacro:if value="${gripper != ''}">
+    <!-- name of the gripper -->
+    <xacro:property name="gripper_name" value="$(arg robot_prefix)gripper"/>
+    <!-- load gripper macro -->
+    <xacro:include filename="$(find moveit_resources_prbt_${gripper}_support)/urdf/${gripper}.urdf.xacro" />
+    <!-- instantiate gripper -->
+    <xacro:prbt_gripper parent="$(arg robot_prefix)flange" />
+    <!-- Add gripper brackets -->
+    <xacro:include filename="$(find moveit_resources_prbt_support)/urdf/simple_gripper_brackets.urdf.xacro" />
+    <xacro:simple_gripper_brackets />
+  </xacro:if>
+</robot>
