Commit message: fixe ik problems & editing the urdf

File: install/moveit_resources_prbt_support/share/moveit_resources_prbt_support/urdf/prbt_macro.xacro (robot description, xacro)
@@ -1 +1,408 @@
-/home/saber/robox_ws/src/moveit2/moveit_planners/test_configs/prbt_support/urdf/prbt_macro.xacro
+<?xml version="1.0" encoding="utf-8" ?>
+<!--
+Copyright (c) 2018 Pilz GmbH & Co. KG
+Licensed under the Apache License, Version 2.0 (the "License");
+you may not use this file except in compliance with the License.
+You may obtain a copy of the License at
+    http://www.apache.org/licenses/LICENSE-2.0
+Unless required by applicable law or agreed to in writing, software
+distributed under the License is distributed on an "AS IS" BASIS,
+WITHOUT WARRANTIES OR CONDITIONS OF ANY KIND, either express or implied.
+See the License for the specific language governing permissions and
+limitations under the License.
+-->
+<robot xmlns:xacro="http://www.ros.org/wiki/xacro">
+  <xacro:macro name="prbt" params="
+    prefix
+    initial_positions:=${dict(joint_1=0.0,joint_2=0.0,joint_3=0.0,joint_4=0.0,joint_5=0.0,joint_6=0.0)}">
+    <!-- Height of Foot -->
+    <xacro:property name="L0" value="0.2604" />
+    <!-- Length of the first connector -->
+    <xacro:property name="L1" value="0.3500" />
+    <!-- Length of the second connector -->
+    <xacro:property name="L2" value="0.3070" />
+    <!-- Distance last joint to flange -->
+    <xacro:property name="L3" value="0.0840" />
+    <!-- ros2 control include -->
+    <xacro:include filename="$(find moveit_resources_prbt_support)/urdf/prbt.ros2_control.xacro" />
+    <!-- ros2 control instance -->
+    <xacro:prbt_ros2_control
+      name="PRBTPositionHardwareInterface" prefix="${prefix}"
+      use_fake_hardware="true"
+      initial_positions="${initial_positions}"
+      fake_sensor_commands="true"/>
+    <!-- robot foot link -->
+    <link name="${prefix}base_link">
+        <inertial>
+          <mass value="2.4"/>
+          <inertia ixx="0"  ixy="0"  ixz="0" iyy="0" iyz="0" izz="0" />
+        </inertial>
+      <visual>
+        <origin xyz="0 0 0" rpy="0 0 0" />
+        <geometry>
+          <mesh filename="package://moveit_resources_prbt_support/meshes/foot.dae" />
+        </geometry>
+      </visual>
+      <collision>
+        <origin rpy="${pi} 0 0" xyz="0 0 0.065"/>
+        <geometry>
+          <cylinder length="0.13" radius="0.09275"/>
+        </geometry>
+      </collision>
+    </link>
+    <!-- arm 1 joint -->
+    <joint name="${prefix}joint_1" type="revolute">
+      <origin xyz="0 0 ${L0}" rpy="0 0 -${pi}"/>
+      <parent link="${prefix}base_link"/>
+      <child link="${prefix}link_1"/>
+      <axis xyz="0 0 1"/>
+      <limit effort="370" velocity="1.57" lower="-2.96706" upper="2.96706"/>
+      <dynamics damping="15.0" friction="11" />
+    </joint>
+    <!-- arm 1 link -->
+    <link name="${prefix}link_1">
+      <inertial>
+        <mass value="7.1"/>
+        <origin xyz="0 -0.026 -0.051" />
+        <inertia ixx="3.53e-2" ixy="0" ixz="0" iyy="3.01e-2" iyz="9.04e-3" izz="1.87e-2" />
+      </inertial>
+      <visual>
+        <origin xyz="0 0 0" rpy="0 0 0" />
+        <geometry>
+          <mesh filename="package://moveit_resources_prbt_support/meshes/link_1.dae" />
+        </geometry>
+      </visual>
+      <collision>
+        <origin rpy="0 0 0" xyz="0 0 -0.08"/>
+        <geometry>
+          <cylinder length="0.10" radius="0.07"/>
+        </geometry>
+      </collision>
+      <collision>
+        <origin rpy="0 0 0" xyz="0 0 0"/>
+        <geometry>
+          <sphere radius="0.09"/>
+        </geometry>
+      </collision>
+      <collision>
+        <origin rpy="0 ${pi/2} ${pi/2}" xyz="0 -0.10 0"/>
+        <geometry>
+          <cylinder length="0.10" radius="0.065"/>
+        </geometry>
+      </collision>
+    </link>
+    <!-- joint between arm_1_link and arm_2_link -->
+    <joint name="${prefix}joint_2" type="revolute">
+      <origin xyz="0 0 0" rpy="${pi/2} 0 0"/>
+      <parent link="${prefix}link_1"/>
+      <child link="${prefix}link_2"/>
+      <axis xyz="0 0 1"/>
+      <limit effort="370" velocity="1.57" lower="-2.53073" upper="2.53073"/>
+      <dynamics damping="12.0" friction="10.0" />
+    </joint>
+    <link name="${prefix}link_2">
+      <inertial>
+        <mass value="1.7"/>
+        <origin xyz="0 0.162 0.134" />
+        <inertia ixx="3.58e-2"  ixy="0"  ixz="0" iyy="3.22e-3" iyz="-1.45e-3" izz="3.66e-2" />
+      </inertial>
+      <visual name="first">
+        <origin xyz="0 0 0" rpy="0 0 0" />
+        <geometry>
+          <mesh filename="package://moveit_resources_prbt_support/meshes/link_2.dae" />
+        </geometry>
+      </visual>
+      <collision>
+        <origin rpy="${pi/18} 0 0" xyz="0 0.15 0.145"/>
+        <geometry>
+          <box size="0.121 0.27 0.065"/>
+        </geometry>
+      </collision>
+      <collision>
+        <origin rpy="-${pi/7} 0 0" xyz="0 0.3 0.145"/>
+        <geometry>
+          <box size="0.11 0.1 0.075"/>
+        </geometry>
+      </collision>
+    </link>
+    <!-- joint between arm_2_link and arm_3_link -->
+    <joint name="${prefix}joint_3" type="revolute">
+      <origin xyz="0 ${L1} 0" rpy="0 ${pi} 0"/>
+      <parent link="${prefix}link_2"/>
+      <child link="${prefix}link_3"/>
+      <axis xyz="0 0 1"/>
+      <limit effort="176" velocity="1.57" lower="-2.35620" upper="2.35620"/>
+      <dynamics damping="4.5" friction="4.5" />
+    </joint>
+    <link name="${prefix}link_3">
+      <inertial>
+        <mass value="4.8"/>
+        <origin xyz="0 0.043 -0.027" />
+        <inertia ixx="2.06e-2" ixy="0" ixz="0" iyy="1.08e-2" iyz="-5.36e-3" izz="1.63e-2" />
+      </inertial>
+      <visual>
+        <origin xyz="0 0 0" rpy="0 0 0" />
+        <geometry>
+          <mesh filename="package://moveit_resources_prbt_support/meshes/link_3.dae" />
+        </geometry>
+      </visual>
+      <collision>
+        <origin rpy="0 0 0" xyz="0 0 -0.11"/>
+        <geometry>
+          <cylinder length="0.10" radius="0.06"/>
+        </geometry>
+      </collision>
+      <collision>
+        <origin rpy="0 0 0" xyz="0 0 0"/>
+        <geometry>
+          <sphere radius="0.085"/>
+        </geometry>
+      </collision>
+      <collision>
+        <origin rpy="0 ${pi/2} ${pi/2}" xyz="0 0.10 0"/>
+        <geometry>
+          <cylinder length="0.10" radius="0.065"/>
+        </geometry>
+      </collision>
+    </link>
+    <!-- joint between arm_3_link and arm_4_link -->
+    <joint name="${prefix}joint_4" type="revolute">
+      <origin xyz="0 0 0" rpy="-${pi/2} ${pi} 0" />
+      <parent link="${prefix}link_3"/>
+      <child link="${prefix}link_4"/>
+      <axis xyz="0 0 1" />
+      <limit effort="176" velocity="1.57" lower="-2.96706" upper="2.96706"/>
+      <dynamics damping="4.2" friction="3.8" />
+    </joint>
+    <link name="${prefix}link_4">
+      <inertial>
+        <mass value="0.9"/>
+        <origin xyz="0 -0.061 0.204" />
+        <inertia ixx="6.79e-3" ixy="0" ixz="0" iyy="4.91e-3" iyz="2.67e-3" izz="3.40e-3" />
+      </inertial>
+      <visual>
+        <origin xyz="0 0 0" rpy="0 0 0" />
+        <geometry>
+          <mesh filename="package://moveit_resources_prbt_support/meshes/link_4.dae" />
+        </geometry>
+      </visual>
+      <collision>
+        <origin rpy="${pi/3.25} 0 0" xyz="0 -0.04 0.162"/>
+        <geometry>
+          <box size="0.121 0.08 0.17"/>
+        </geometry>
+      </collision>
+      <collision>
+        <origin rpy="-${pi/30} 0 0" xyz="0 -0.115 0.25"/>
+        <geometry>
+          <box size="0.09 0.06 0.12"/>
+        </geometry>
+      </collision>
+    </link>
+    <!-- joint between arm_4_link and arm_5_link -->
+    <joint name="${prefix}joint_5" type="revolute">
+      <origin xyz="0 0 ${L2}" rpy="${pi/2} 0 ${pi}" />
+      <parent link="${prefix}link_4"/>
+      <child link="${prefix}link_5"/>
+      <axis xyz="0 0 1" />
+      <limit effort="41.6" velocity="1.57" lower="-2.96706" upper="2.96706" />
+      <dynamics damping="1.5" friction="3.5" />
+    </joint>
+    <link name="${prefix}link_5">
+      <inertial>
+        <mass value="2.6"/>
+        <origin xyz="-0.001 0.021 -0.032" />
+        <inertia ixx="7.37e-3" ixy="4.78e-6" ixz="6.00e-5" iyy="5.87e-3" iyz="-1.71e-3" izz="3.96e-3" />
+      </inertial>
+      <visual>
+        <origin xyz="0 0 0" rpy="0 0 0" />
+        <geometry>
+          <mesh filename="package://moveit_resources_prbt_support/meshes/link_5.dae"/>
+        </geometry>
+      </visual>
+      <collision>
+        <origin rpy="0 0 0" xyz="0 0 -0.095"/>
+        <geometry>
+          <cylinder length="0.08" radius="0.045"/>
+        </geometry>
+      </collision>
+      <collision>
+        <origin rpy="0 0 0" xyz="0 0 -0.06"/>
+        <geometry>
+          <cylinder length="0.04" radius="0.0545"/>
+        </geometry>
+      </collision>
+      <collision>
+        <origin rpy="0 0 0" xyz="0 0 0"/>
+        <geometry>
+          <sphere radius="0.07"/>
+        </geometry>
+      </collision>
+      <collision>
+        <origin rpy="0 ${pi/2} ${pi/2}" xyz="0 0.05 0"/>
+        <geometry>
+          <cylinder length="0.03" radius="0.05"/>
+        </geometry>
+      </collision>
+      <collision>
+        <origin rpy="0 ${pi/2} ${pi/2}" xyz="0 0.05 0"/>
+        <geometry>
+          <cylinder length="0.049" radius="0.0435"/>
+        </geometry>
+      </collision>
+    </link>
+    <!-- joint between arm_5_link and flange -->
+    <joint name="${prefix}joint_6" type="revolute">
+      <origin xyz="0 ${L3} 0" rpy="-${pi/2} 0 0" />
+      <parent link="${prefix}link_5"/>
+      <child link="${prefix}flange"/>
+      <axis xyz="0 0 1" />
+      <limit effort="20.1" velocity="1.57" lower="-3.12414" upper="3.12414" />
+      <dynamics damping="4.5" friction="7.0" />
+    </joint>
+    <!-- Flange -->
+    <link name="${prefix}flange">
+      <inertial>
+        <mass value="0.02" />
+        <origin xyz="0 0 0" />
+        <inertia ixx="0" ixy="0" ixz="0" iyy="0" iyz="0" izz="0" />
+      </inertial>
+      <visual>
+        <origin xyz="0 0 0" rpy="0 0 0" />
+        <geometry>
+          <mesh filename="package://moveit_resources_prbt_support/meshes/flange.dae"/>
+        </geometry>
+      </visual>
+      <collision>
+        <origin rpy="0 0 0" xyz="0 0 -0.0035"/>
+        <geometry>
+          <cylinder length="0.02" radius="0.0331"/>
+        </geometry>
+      </collision>
+    </link>
+    <!-- ROS-Industrial 'base' frame: base_link to robot world coordinate system transform -->
+    <link name="${prefix}base" />
+    <joint name="${prefix}base_link-base" type="fixed">
+      <origin xyz="0 0 0" rpy="0 0 0"/>
+      <parent link="${prefix}base_link"/>
+      <child link="${prefix}base"/>
+    </joint>
+    <!-- ROS-Industrial 'tool0' frame: all-zeros tool frame -->
+    <link name="${prefix}tool0" />
+    <joint name="${prefix}flange-tool0" type="fixed">
+      <origin xyz="0 0 0" rpy="0 0 0" />
+      <parent link="${prefix}flange" />
+      <child link="${prefix}tool0" />
+    </joint>
+    <!-- transmissions for gazebo -->
+    <transmission name="${prefix}joint_1_trans">
+      <type>transmission_interface/SimpleTransmission</type>
+      <joint name="${prefix}joint_1">
+        <hardwareInterface>hardware_interface/PositionJointInterface</hardwareInterface>
+      </joint>
+      <actuator name="${prefix}joint_1_motor"/>
+    </transmission>
+    <transmission name="${prefix}joint_2_trans">
+      <type>transmission_interface/SimpleTransmission</type>
+      <joint name="${prefix}joint_2">
+        <hardwareInterface>hardware_interface/PositionJointInterface</hardwareInterface>
+      </joint>
+      <actuator name="${prefix}joint_2_motor"/>
+    </transmission>
+    <transmission name="${prefix}joint_3_trans">
+      <type>transmission_interface/SimpleTransmission</type>
+      <joint name="${prefix}joint_3">
+        <hardwareInterface>hardware_interface/PositionJointInterface</hardwareInterface>
+      </joint>
+      <actuator name="${prefix}joint_3_motor"/>
+    </transmission>
+    <transmission name="${prefix}joint_4_trans">
+      <type>transmission_interface/SimpleTransmission</type>
+      <joint name="${prefix}joint_4">
+        <hardwareInterface>hardware_interface/PositionJointInterface</hardwareInterface>
+      </joint>
+      <actuator name="${prefix}joint_4_motor"/>
+    </transmission>
+    <transmission name="${prefix}joint_5_trans">
+      <type>transmission_interface/SimpleTransmission</type>
+      <joint name="${prefix}joint_5">
+        <hardwareInterface>hardware_interface/PositionJointInterface</hardwareInterface>
+      </joint>
+      <actuator name="${prefix}joint_5_motor"/>
+    </transmission>
+    <transmission name="${prefix}joint_6_trans">
+      <type>transmission_interface/SimpleTransmission</type>
+      <joint name="${prefix}joint_6">
+        <hardwareInterface>hardware_interface/PositionJointInterface</hardwareInterface>
+      </joint>
+      <actuator name="${prefix}joint_6_motor"/>
+    </transmission>
+    <gazebo>
+      <plugin name="gazebo_ros_control" filename="libgazebo_ros_control.so" >
+        <robotNamespace>prbt</robotNamespace>
+        <robotSimType>gazebo_ros_control/DefaultRobotHWSim</robotSimType>
+        <legacyModeNS>false</legacyModeNS> <!-- Only used from ros-kinetic-gazebo-ros-control 2.5.18 -->
+      </plugin>
+    </gazebo>
+    <gazebo reference="${prefix}joint_1">
+      <provideFeedback>true</provideFeedback>
+    </gazebo>
+    <gazebo>
+      <plugin name="ft_sensor" filename="libgazebo_ros_ft_sensor.so">
+	<updateRate>100.0</updateRate>
+	<topicName>prbt/ft_sensor/joint_1</topicName>
+	<jointName>${prefix}joint_1</jointName>
+      </plugin>
+    </gazebo>
+    <gazebo reference="${prefix}joint_2">
+      <provideFeedback>true</provideFeedback>
+    </gazebo>
+    <gazebo>
+      <plugin name="ft_sensor" filename="libgazebo_ros_ft_sensor.so">
+	<updateRate>100.0</updateRate>
+	<topicName>prbt/ft_sensor/joint_2</topicName>
+	<jointName>${prefix}joint_2</jointName>
+      </plugin>
+    </gazebo>
+    <gazebo reference="${prefix}joint_3">
+      <provideFeedback>true</provideFeedback>
+    </gazebo>
+    <gazebo>
+      <plugin name="ft_sensor" filename="libgazebo_ros_ft_sensor.so">
+	<updateRate>100.0</updateRate>
+	<topicName>prbt/ft_sensor/joint_3</topicName>
+	<jointName>${prefix}joint_3</jointName>
+      </plugin>
+    </gazebo>
+    <gazebo reference="${prefix}joint_4">
+      <provideFeedback>true</provideFeedback>
+    </gazebo>
+    <gazebo>
+      <plugin name="ft_sensor" filename="libgazebo_ros_ft_sensor.so">
+	<updateRate>100.0</updateRate>
+	<topicName>prbt/ft_sensor/joint_4</topicName>
+	<jointName>${prefix}joint_4</jointName>
+      </plugin>
+    </gazebo>
+    <gazebo reference="${prefix}joint_5">
+      <provideFeedback>true</provideFeedback>
+    </gazebo>
+    <gazebo>
+      <plugin name="ft_sensor" filename="libgazebo_ros_ft_sensor.so">
+	<updateRate>100.0</updateRate>
+	<topicName>prbt/ft_sensor/joint_5</topicName>
+	<jointName>${prefix}joint_5</jointName>
+      </plugin>
+    </gazebo>
+    <gazebo reference="${prefix}joint_6">
+      <provideFeedback>true</provideFeedback>
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
File: install/moveit_resources_prbt_support/share/moveit_resources_prbt_support/urdf/simple_gripper_brackets.urdf.xacro (robot description, xacro)
@@ -1 +1,85 @@
-/home/saber/robox_ws/src/moveit2/moveit_planners/test_configs/prbt_support/urdf/simple_gripper_brackets.urdf.xacro
+<?xml version="1.0" ?>
+<!--
+Copyright (c) 2018 Pilz GmbH & Co. KG
+Licensed under the Apache License, Version 2.0 (the "License");
+you may not use this file except in compliance with the License.
+You may obtain a copy of the License at
+    http://www.apache.org/licenses/LICENSE-2.0
+Unless required by applicable law or agreed to in writing, software
+distributed under the License is distributed on an "AS IS" BASIS,
+WITHOUT WARRANTIES OR CONDITIONS OF ANY KIND, either express or implied.
+See the License for the specific language governing permissions and
+limitations under the License.
+-->
+<robot xmlns:xacro="http://www.ros.org/wiki/xacro">
+  <xacro:macro name="simple_gripper_brackets"
+               params="gripper_name:=^
+                       parent_left:=^|''
+                       parent_right:=^|''
+                       size_x:=^|0.03
+                       size_y:=^|0.01
+                       size_z:=^|0.05">
+    <xacro:if value="${parent_left==''}">
+      <xacro:property name="parent_left" value="${gripper_name}_finger_left_link" />
+    </xacro:if>
+    <xacro:if value="${parent_right==''}">
+      <xacro:property name="parent_right" value="${gripper_name}_finger_right_link" />
+    </xacro:if>
+    <!-- fixed joint attaching to left bracket mounting -->
+    <joint name="${gripper_name}_link_left_bracket_fixed_joint" type="fixed">
+      <parent link="${parent_left}"/>
+      <child link="${gripper_name}_finger_left_link_bracket"/>
+    </joint>
+    <!-- link of left bracket -->
+    <link name="${gripper_name}_finger_left_link_bracket">
+        <inertial>
+          <origin xyz="0 0 0" rpy="0 0 0"/>
+          <mass value="1"/>
+          <inertia ixx="0.01" ixy="0" ixz="0" iyy="0.01" iyz="0" izz="0.01" />
+        </inertial>
+        <visual>
+          <origin xyz="0 ${size_y/2} ${size_z/2-0.005}" rpy="0 0 0" />
+          <geometry>
+            <box size="${size_x} ${size_y} ${size_z}"/>
+          </geometry>
+          <material name="light_gray">
+            <color rgba="0.6 0.6 0.6 1"/>
+          </material>
+        </visual>
+        <collision>
+          <origin xyz="0 ${size_y/2} ${size_z/2-0.005}" rpy="0 0 0" />
+          <geometry>
+            <box size="${size_x} ${size_y} ${size_z}"/>
+          </geometry>
+        </collision>
+    </link>
+    <!-- fixed joint attaching to right bracket mounting -->
+    <joint name="${gripper_name}_link_right_bracket_fixed_joint" type="fixed">
+      <parent link="${parent_right}"/>
+      <child link="${gripper_name}_finger_right_link_bracket"/>
+    </joint>
+    <!-- link of right bracket -->
+    <link name="${gripper_name}_finger_right_link_bracket">
+        <inertial>
+          <origin xyz="0 0 0" rpy="0 0 0"/>
+          <mass value="1"/>
+          <inertia ixx="0.01" ixy="0" ixz="0" iyy="0.01" iyz="0" izz="0.01" />
+        </inertial>
+        <visual>
+          <origin xyz="0 -${size_y/2} ${size_z/2-0.005}" rpy="0 0 0" />
+          <geometry>
+            <box size="${size_x} ${size_y} ${size_z}"/>
+          </geometry>
+          <material name="dark_grey">
+            <color rgba="0.8 0.8 0.8 1"/>
+          </material>
+        </visual>
+        <collision>
+          <origin xyz="0 -${size_y/2} ${size_z/2-0.005}" rpy="0 0 0" />
+          <geometry>
+            <box size="${size_x} ${size_y} ${size_z}"/>
+          </geometry>
+        </collision>
+    </link>
+  </xacro:macro>
+</robot>
