Commit message: pick and place pub/sub approach

File: src/robox_arm/urdf/robox_arm.urdf (robot description, URDF)
Before this commit: robot robox_arm, 9 links, 8 joints
Links:
- added link ik_frame, mass 0.001
Joints:
- added joint link_five_to_ik_frame: type fixed, parent link_five, child ik_frame, origin xyz=-0.01 0.0 0.1 rpy=0 0 0
- joint joint_seven: axis 0 -0.994576407261666 -0.104008509836822 -> 0 -1 0; limit lower=-0.03 upper=0 effort=1 velocity=1.0 -> lower=-1.221 upper=0.097 effort=1 velocity=1.0
- joint joint_six: axis 0 0.99457640726172 -0.104008509836308 -> 0 1 0; limit lower=-0.03 upper=0 effort=1 velocity=1.0 -> lower=-1.221 upper=0.097 effort=1 velocity=1.0
- joint joint_two: limit lower=-1.57 upper=0.69 effort=100 velocity=1.0 -> lower=-1.307 upper=0.617 effort=100 velocity=1.0
- joint world_to_base: origin xyz=0 0 0 rpy=0 0 0 -> xyz= -0.09191  0.125 -0.015 rpy=0 0 0

Commit message: pick and place using action server/client

File: src/robox_arm/urdf/robox_arm.urdf (robot description, URDF)
Before this commit: robot robox_arm, 10 links, 9 joints
Joints:
- joint joint_five: origin xyz=0.00975000000002091 -0.0263999999999991 0.0726000000000027 rpy=0 0 0 -> xyz=0.01 -0.0264 0.0726000000000027 rpy=0 0 0
- joint joint_one: origin xyz=0 0 0.0466 rpy=0 0 0 -> xyz=0 0 0.04444 rpy=0 0 0
- joint joint_three: origin xyz=0 0.000700000000000298 0.100000000000001 rpy=0 0 0 -> xyz=0 0.0 0.100000000000001 rpy=0 0 0
- joint joint_two: origin xyz=0.00949999999999964 0.0247000000000005 0.03197 rpy=0 0 0 -> xyz=0.00949999999999964 0.0247 0.03282 rpy=0 0 0
- joint link_five_to_ik_frame: origin xyz=-0.01 0.0 0.1 rpy=0 0 0 -> xyz=0.0 0.0 0.0954 rpy=0 0 0
- joint world_to_base: origin xyz= -0.09191  0.125 -0.015 rpy=0 0 0 -> xyz= -0.09191  0.125 -0.0135 rpy=0 0 0
