Commit message: Adding GUI that contains 5 Modes

File: install/robox_moveit_config/share/robox_moveit_config/config/robox_arm.ros2_control.xacro (robot description, xacro)
@@ -1,59 +1 @@
-<?xml version="1.0"?>
-<robot xmlns:xacro="http://www.ros.org/wiki/xacro">
-  <xacro:macro name="robox_arm_ros2_control" params="name initial_positions_file">
-    <ros2_control name="${name}" type="system">
-      <hardware>
-        <plugin>mock_components/GenericSystem</plugin>
-      </hardware>
-      <joint name="joint_one">
-        <command_interface name="position"/>
-        <state_interface name="position">
-          <param name="initial_value">0.0</param>
-        </state_interface>
-        <state_interface name="velocity"/>
-      </joint>
-      <joint name="joint_two">
-        <command_interface name="position"/>
-        <state_interface name="position">
-          <param name="initial_value">0.0</param>
-        </state_interface>
-        <state_interface name="velocity"/>
-      </joint>
-      <joint name="joint_three">
-        <command_interface name="position"/>
-        <state_interface name="position">
-          <param name="initial_value">0.0</param>
-        </state_interface>
-        <state_interface name="velocity"/>
-      </joint>
-      <joint name="joint_four">
-        <command_interface name="position"/>
-        <state_interface name="position">
-          <param name="initial_value">0.0</param>
-        </state_interface>
-        <state_interface name="velocity"/>
-      </joint>
-      <joint name="joint_five">
-        <command_interface name="position"/>
-        <state_interface name="position">
-          <param name="initial_value">0.0</param>
-        </state_interface>
-        <state_interface name="velocity"/>
-      </joint>
-      <joint name="joint_six">
-        <command_interface name="position"/>
-        <state_interface name="position">
-          <param name="initial_value">0.0</param>
-        </state_interface>
-        <state_interface name="velocity"/>
-      </joint>
-      <joint name="joint_seven">
-        <command_interface name="position"/>
-        <state_interface name="position">
-          <param name="initial_value">0.0</param>
-        </state_interface>
-        <state_interface name="velocity"/>
-      </joint>
-    </ros2_control>
-  </xacro:macro>
-</robot>
+/home/saber/robox_ws/src/robox_moveit_config/config/robox_arm.ros2_control.xacro

File: install/robox_moveit_config/share/robox_moveit_config/config/robox_arm.urdf.xacro (robot description, xacro)
@@ -1,9 +1 @@
-<?xml version="1.0"?>
-<robot xmlns:xacro="http://www.ros.org/wiki/xacro" name="robox_arm">
-    <xacro:arg name="initial_positions_file" default="initial_positions.yaml" />
-    <!-- Import robox_arm urdf file -->
-    <xacro:include filename="$(find robox_arm)/urdf/robox_arm.urdf" />
-    <!-- Import control_xacro -->
-    <xacro:include filename="robox_arm.ros2_control.xacro" />
-    <xacro:robox_arm_ros2_control name="FakeSystem" initial_positions_file="$(arg initial_positions_file)"/>
-</robot>
+/home/saber/robox_ws/src/robox_moveit_config/config/robox_arm.urdf.xacro

File: src/install/robox_arm/share/robox_arm/urdf/robox_arm.urdf (robot description, URDF)
Before this commit: robot robox_arm, 10 links, 9 joints
Joints:
- joint joint_five: origin xyz=0.00975000000002091 -0.0263999999999991 0.0726000000000027 rpy=0 0 0 -> xyz=0.01 -0.0264 0.0726000000000027 rpy=0 0 0
- joint joint_one: origin xyz=0 0 0.0466 rpy=0 0 0 -> xyz=0 0 0.04444 rpy=0 0 0
- joint joint_three: origin xyz=0 0.000700000000000298 0.100000000000001 rpy=0 0 0 -> xyz=0 0.0 0.100000000000001 rpy=0 0 0
- joint joint_two: origin xyz=0.00949999999999964 0.0247000000000005 0.03197 rpy=0 0 0 -> xyz=0.00949999999999964 0.0247 0.03282 rpy=0 0 0
- joint link_five_to_ik_frame: origin xyz=-0.015 0.0 0.1 rpy=0 0 0 -> xyz=0.0 0.0 0.0954 rpy=0 0 0
- joint world_to_base: origin xyz= -0.09191  0.125 -0.015 rpy=0 0 0 -> xyz= -0.09191  0.125 -0.0135 rpy=0 0 0

Commit message: color stacking mode is adjusted and the front end of the GUI is enhanced

File: install/robox_moveit_config/share/robox_moveit_config/config/robox_arm.ros2_control.xacro (robot description, xacro)
@@ -1 +1,59 @@
-/home/saber/robox_ws/src/robox_moveit_config/config/robox_arm.ros2_control.xacro
+<?xml version="1.0"?>
+<robot xmlns:xacro="http://www.ros.org/wiki/xacro">
+  <xacro:macro name="robox_arm_ros2_control" params="name initial_positions_file">
+    <ros2_control name="${name}" type="system">
+      <hardware>
+        <plugin>mock_components/GenericSystem</plugin>
+      </hardware>
+      <joint name="joint_one">
+        <command_interface name="position"/>
+        <state_interface name="position">
+          <param name="initial_value">0.0</param>
+        </state_interface>
+        <state_interface name="velocity"/>
+      </joint>
+      <joint name="joint_two">
+        <command_interface name="position"/>
+        <state_interface name="position">
+          <param name="initial_value">0.0</param>
+        </state_interface>
+        <state_interface name="velocity"/>
+      </joint>
+      <joint name="joint_three">
+        <command_interface name="position"/>
+        <state_interface name="position">
+          <param name="initial_value">0.0</param>
+        </state_interface>
+        <state_interface name="velocity"/>
+      </joint>
+      <joint name="joint_four">
+        <command_interface name="position"/>
+        <state_interface name="position">
+          <param name="initial_value">0.0</param>
+        </state_interface>
+        <state_interface name="velocity"/>
+      </joint>
+      <joint name="joint_five">
+        <command_interface name="position"/>
+        <state_interface name="position">
+          <param name="initial_value">0.0</param>
+        </state_interface>
+        <state_interface name="velocity"/>
+      </joint>
+      <joint name="joint_six">
+        <command_interface name="position"/>
+        <state_interface name="position">
+          <param name="initial_value">0.0</param>
+        </state_interface>
+        <state_interface name="velocity"/>
+      </joint>
+      <joint name="joint_seven">
+        <command_interface name="position"/>
+        <state_interface name="position">
+          <param name="initial_value">0.0</param>
+        </state_interface>
+        <state_interface name="velocity"/>
+      </joint>
+    </ros2_control>
+  </xacro:macro>
+</robot>

File: install/robox_moveit_config/share/robox_moveit_config/config/robox_arm.urdf.xacro (robot description, xacro)
@@ -1 +1,9 @@
-/home/saber/robox_ws/src/robox_moveit_config/config/robox_arm.urdf.xacro
+<?xml version="1.0"?>
+<robot xmlns:xacro="http://www.ros.org/wiki/xacro" name="robox_arm">
+    <xacro:arg name="initial_positions_file" default="initial_positions.yaml" />
+    <!-- Import robox_arm urdf file -->
+    <xacro:include filename="$(find robox_arm)/urdf/robox_arm.urdf" />
+    <!-- Import control_xacro -->
+    <xacro:include filename="robox_arm.ros2_control.xacro" />
+    <xacro:robox_arm_ros2_control name="FakeSystem" initial_positions_file="$(arg initial_positions_file)"/>
+</robot>

File: src/robox_arm/urdf/robox_arm.urdf (robot description, URDF)
Before this commit: robot robox_arm, 10 links, 9 joints
Joints:
- joint world_to_base: origin xyz= -0.09191  0.125 -0.0135 rpy=0 0 0 -> xyz= -0.092  0.100 -0.0135 rpy=0 0 0
